File: GT-Wheel-RevLight/GT-Wheel-RevLight.kicad_sch (KiCad schematic)
At the start: 82 parts, among them SW1 SKSTAJE010, SW2 SKSTAJE010, SW3 SKSTAJE010, SW4 SKSTAJE010, SW5 SKSTAJE010, SW6 SKSTAJE010

Commit message: routing done
Parts:
- added C23, C24, C25, C26, C27, C28: 100nF-CER-25V-0402, Capacitor_SMD:C_0402_1005Metric, symbol CAP-SMD-25V:100nF-CER-25V-0402
- added D25, D26, D27, D28, D29, D30: WS2812B, LED_SMD:LED_WS2812B_PLCC4_5.0x5.0mm_P3.2mm, symbol LED:WS2812B
- renumbered D13 to D10, D15 to D11, D17 to D12, D19 to D13, D21 to D14, D23 to D15, D25 to D16, D8 to D17, D10 to D18, D12 to D19, D14 to D20, D16 to D21, D18 to D22, D20 to D23, D22 to D24, D9 to D8, D11 to D9
Connections:
- net LOGIC_GND: now also C23.2, C24.2, C25.2, C26.2, C27.2, C28.2, D25.3 (VSS), D26.3 (VSS), D27.3 (VSS), D28.3 (VSS), D29.3 (VSS), D30.3 (VSS)
- net +5V: now reaches C3.1, D8.1 (VDD)
- net +5V: now also C1.1, C10.1, C11.1, C12.1, C13.1, C14.1, C15.1, C16.1, C17.1, C19.1, C2.1, C4.1, C5.1, C6.1, C7.1, C8.1, C9.1, D10.1 (VDD), D11.1 (VDD), D12.1 (VDD), D13.1 (VDD), D14.1 (VDD), D15.1 (VDD), D16.1 (VDD), D17.1 (VDD), D18.1 (VDD), D19.1 (VDD), D20.1 (VDD), D21.1 (VDD), D22.1 (VDD), D23.1 (VDD), D24.1 (VDD), D7.1 (VDD), D9.1 (VDD), WP20.1, C23.1, C24.1, C25.1, C26.1, C27.1, C28.1, D25.1 (VDD), D26.1 (VDD), D27.1 (VDD), D28.1 (VDD), D29.1 (VDD), D30.1 (VDD)
- net at D24.2 (DOUT): now also D25.4 (DIN)
- net +3.3V: now reaches R3.1, R4.1
- net +3.3V: now also R7.1, R8.1, WP22.1
- new net: D25.2 (DOUT), D26.4 (DIN)
- new net: D28.2 (DOUT), D29.4 (DIN)
- new net: D27.2 (DOUT), D28.4 (DIN)
- new net: D29.2 (DOUT), D30.4 (DIN)
- new net: D26.2 (DOUT), D27.4 (DIN)
- no-connect marks 1 -> 0
Other:
- moved on the sheet: C1, C10, C11, C12, C13, C14, C15, C16, C17, C19, C2, C3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
