File: GT-Wheel-Main-PCB/GT-Wheel.kicad_pcb (KiCad board)
At the start: 2 copper layers, 157 parts, among them J2 TC2050, J3 0532610471, J4 USB_A, J5 0532610871, J6 0532610871, SW1 56DP30-01-1-AJN, SW10 SKSTAJE010, SW2 56DP30-01-1-AJN, SW3 56DP30-01-1-AJN, SW4 56DP30-01-1-AJN, SW5 SKSTAJE010, SW6 SKSTAJE010, SW7 SKSTAJE010, SW8 SKSTAJE010, SW9 SKSTAJE010, U1 STM32F303RETx, U2 USB2512B, U3 AP2112K-3.3, X1 8MHz, X2 24MHz

Commit message: removing usb hub
Parts:
- removed SW10, SW9: SKSTAJE010, SWITCH-SMD-TACTILE:SKSTAJE010
- added C56: 100nF-CER-25V-0402, Capacitor_SMD:C_0402_1005Metric, F.Cu at (350.5, 44.6)
- added C57: 100nF-CER-25V-0402, Capacitor_SMD:C_0402_1005Metric, F.Cu at (353.4, 28.8)
- added C58: 100nF-CER-25V-0402, Capacitor_SMD:C_0402_1005Metric, F.Cu at (353.4, 30.8)
- added C59: 100nF-CER-25V-0402, Capacitor_SMD:C_0402_1005Metric, F.Cu at (353.4, 32.8)
- added C60: 100nF-CER-25V-0402, Capacitor_SMD:C_0402_1005Metric, F.Cu at (353.4, 34.7)
- added C61: 100nF-CER-25V-0402, Capacitor_SMD:C_0402_1005Metric, F.Cu at (353.4, 36.7)
- added C62: 100nF-CER-25V-0402, Capacitor_SMD:C_0402_1005Metric, F.Cu at (353.4, 38.7)
- added C63: 100nF-CER-25V-0402, Capacitor_SMD:C_0402_1005Metric, F.Cu at (353.4, 40.6)
- added C64: 100nF-CER-25V-0402, Capacitor_SMD:C_0402_1005Metric, F.Cu at (346.7, 108.2)
- added C65: 100nF-CER-25V-0402, Capacitor_SMD:C_0402_1005Metric, F.Cu at (346.7, 110.1)
- added C66: 100nF-CER-25V-0402, Capacitor_SMD:C_0402_1005Metric, F.Cu at (346.7, 112.1)
- added C67: 100nF-CER-25V-0402, Capacitor_SMD:C_0402_1005Metric, F.Cu at (346.7, 114.1)
- added D16: BAT43W-TP, Diode_SMD:D_SOD-123, F.Cu at (309.8, 122.3)
- added D17: BAT43W-TP, Diode_SMD:D_SOD-123, F.Cu at (309.8, 125.7)
- added ENC1: PEC11H-4015F-S0016, SWITCH-THT-ENC:PEC11H-4015F-S0016, F.Cu at (109.2, 102.4)
- added ENC2: PEC11H-4015F-S0016, SWITCH-THT-ENC:PEC11H-4015F-S0016, F.Cu at (129.2, 122.4)
- added ENC3: PEC11H-4015F-S0016, SWITCH-THT-ENC:PEC11H-4015F-S0016, F.Cu at (164.2, 122.4)
- added ENC4: PEC11H-4015F-S0016, SWITCH-THT-ENC:PEC11H-4015F-S0016, F.Cu at (184.2, 102.4)
- added R20: r=663, Resistor_SMD:R_0603_1608Metric, F.Cu at (345.7, 79.8)
- added R21: 10kR-SMD-100mW-0603, Resistor_SMD:R_0603_1608Metric, F.Cu at (349.3, 65.2)
- added R22: 10kR-SMD-100mW-0603, Resistor_SMD:R_0603_1608Metric, F.Cu at (349.3, 67.8)
- added R23: 10kR-SMD-100mW-0603, Resistor_SMD:R_0603_1608Metric, F.Cu at (349.3, 70.3)
- added R24: 10kR-SMD-100mW-0603, Resistor_SMD:R_0603_1608Metric, F.Cu at (349.3, 72.8)
- added R25: 10kR-SMD-100mW-0603, Resistor_SMD:R_0603_1608Metric, F.Cu at (353.3, 60.2)
- added R26: 10kR-SMD-100mW-0603, Resistor_SMD:R_0603_1608Metric, F.Cu at (353.3, 62.7)
- added R27: 10kR-SMD-100mW-0603, Resistor_SMD:R_0603_1608Metric, F.Cu at (353.3, 65.2)
- added R28: 10kR-SMD-100mW-0603, Resistor_SMD:R_0603_1608Metric, F.Cu at (353.3, 67.8)
- added R29: 10kR-SMD-100mW-0603, Resistor_SMD:R_0603_1608Metric, F.Cu at (353.3, 70.3)
- added R30: 10kR-SMD-100mW-0603, Resistor_SMD:R_0603_1608Metric, F.Cu at (353.3, 72.8)
- added R31: 10kR-SMD-100mW-0603, Resistor_SMD:R_0603_1608Metric, F.Cu at (357.3, 60.2)
- added R32: 10kR-SMD-100mW-0603, Resistor_SMD:R_0603_1608Metric, F.Cu at (357.3, 62.7)
- added R33: 10kR-SMD-100mW-0603, Resistor_SMD:R_0603_1608Metric, F.Cu at (357.3, 65.2)
- added R34: 10kR-SMD-100mW-0603, Resistor_SMD:R_0603_1608Metric, F.Cu at (357.3, 67.8)
- added R35: 10kR-SMD-100mW-0603, Resistor_SMD:R_0603_1608Metric, F.Cu at (357.3, 70.3)
- added R36: 10kR-SMD-100mW-0603, Resistor_SMD:R_0603_1608Metric, F.Cu at (357.3, 72.8)
- added R37: 10kR-SMD-100mW-0603, Resistor_SMD:R_0603_1608Metric, F.Cu at (345.7, 82.3)
- added R38: 10kR-SMD-100mW-0603, Resistor_SMD:R_0603_1608Metric, F.Cu at (345.7, 84.8)
- added R39: 10kR-SMD-100mW-0603, Resistor_SMD:R_0603_1608Metric, F.Cu at (345.7, 87.3)
- added R40: 10kR-SMD-100mW-0603, Resistor_SMD:R_0603_1608Metric, F.Cu at (345.7, 89.8)
- added R41: 10kR-SMD-100mW-0603, Resistor_SMD:R_0603_1608Metric, F.Cu at (349.7, 77.3)
- added R42: 10kR-SMD-100mW-0603, Resistor_SMD:R_0603_1608Metric, F.Cu at (349.7, 79.8)
- added R43: 10kR-SMD-100mW-0603, Resistor_SMD:R_0603_1608Metric, F.Cu at (349.7, 82.3)
- added R44: 10kR-SMD-100mW-0603, Resistor_SMD:R_0603_1608Metric, F.Cu at (349.7, 84.8)
- C6, C7: footprint Capacitor_SMD:C_0402_1005Metric -> Capacitor_SMD:C_0201_0603Metric
- SW1, SW2, SW3, SW4: value 56DP30-01-1-AJN -> SKSTAJE010; footprint SWITCH-THT-ROTARY:56DP30-01-1-AJN -> SWITCH-SMD-TACTILE:SKSTAJE010
- SW7, SW8: value SKSTAJE010 -> ~; footprint SWITCH-SMD-TACTILE:SKSTAJE010 -> SWITCH-THT-FUNKY:RKJXT1F42001
- X1: value 8MHz -> 32MHz; footprint Crystal:Crystal_SMD_EuroQuartz_MT-4Pin_3.2x2.5mm -> Crystal:Crystal_SMD_EuroQuartz_X22-4Pin_2.5x2.0mm
- moved WP18 310.0 mm to (363.6, 60.4)
- moved WP19 310.0 mm to (363.6, 63.2)
- moved WP20 310.0 mm to (363.6, 66.1)
- moved WP21 310.0 mm to (363.6, 68.9)
- moved WP22 310.0 mm to (363.6, 71.8)
- moved WP13 310.0 mm to (360.8, 60.4)
- moved WP14 310.0 mm to (360.8, 63.2)
- moved WP15 310.0 mm to (360.8, 66.1)
- moved WP16 310.0 mm to (360.8, 68.9)
- moved WP17 310.0 mm to (360.8, 71.8)
- moved R11 302.1 mm to (349.3, 60.2)
- moved R12 302.1 mm to (349.3, 62.7)
- moved R10 297.9 mm to (345.3, 72.8)
- moved R5 297.9 mm to (345.3, 60.2)
- moved R6 297.9 mm to (345.3, 62.7)
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Connections:
- C7 pad 2: Net-(U1-PF1) -> Net-(C7-Pad2)
- D10 pad 2: /ROW5 -> /ROW2
- D11 pad 2: /ROW5 -> /ROW1
- D12 pad 2: /ROW5 -> /ROW1
- D13 pad 2: /ROW5 -> /ROW1
- D14 pad 2: /ROW6 -> /ROW1
- D15 pad 2: /ROW6 -> /ROW2
- D4 pad 2: /ROW1 -> /ROW3
- D5 pad 2: /ROW2 -> /ROW3
- D7 pad 2: /ROW4 -> /ROW3
- D8 pad 2: /ROW5 -> /ROW2
- D9 pad 2: /ROW5 -> /ROW2
- J5 pad 1: /ROW5 -> Net-(J5-Pad1)
- J5 pad 2: ~ -> /ROW4
- J5 pad 3: /COL7 -> /ROW5
- J5 pad 4: /COL8 -> ~
- J5 pad 5: /COL9 -> /COL1
- J5 pad 6: /COL10 -> /COL2
- J5 pad 7: /COL11 -> /COL3
- J5 pad 8: /COL12 -> ~
- SW1 pad 1: /COL1 -> Net-(D11-K)
- SW1 pad 2: /COL2 -> /COL1
- SW2 pad 1: /COL1 -> Net-(D12-K)
- SW3 pad 1: /COL1 -> Net-(D13-K)
- SW3 pad 2: /COL2 -> /COL3
- SW4 pad 1: /COL1 -> Net-(D8-K)
- SW4 pad 2: /COL2 -> /COL1
- SW5 pad 1: Net-(D8-K) -> Net-(D9-K)
- SW5 pad 2: /COL1 -> /COL2
- SW6 pad 1: Net-(D9-K) -> Net-(D10-K)
- SW6 pad 2: /COL2 -> /COL3
- SW7 pad 1: Net-(D10-K) -> /COL1
- SW7 pad 2: /COL3 -> /COL2
- SW8 pad 1: Net-(D11-K) -> /COL1
- SW8 pad 2: /COL4 -> /COL2
- U1 pad 10: unconnected-(U1-PC2-Pad10) -> /NAV1_ENC_A
- U1 pad 11: unconnected-(U1-PC3-Pad11) -> /NAV1_ENC_B
- U1 pad 2: unconnected-(U1-PC13-Pad2) -> /NAV2_ENC_A
- U1 pad 26: /COL3 -> /ROW6
- U1 pad 27: /COL4 -> /ROW7
- U1 pad 28: /COL5 -> /EN5_A
- U1 pad 3: unconnected-(U1-PC14-Pad3) -> /NAV2_ENC_B
- U1 pad 35: unconnected-(U1-PB14-Pad35) -> /EN8_A
- U1 pad 36: /COL6 -> /EN8_B
- U1 pad 37: /COL7 -> /COL3
- U1 pad 38: /COL8 -> /COL4
- U1 pad 39: /COL9 -> /ROW1
- U1 pad 40: /COL10 -> /ROW2
- U1 pad 41: /COL11 -> unconnected-(U1-PA8-Pad41)
- U1 pad 50: /COL12 -> unconnected-(U1-PA15-Pad50)
- U1 pad 51: /ROW1 -> /ROW3
- U1 pad 52: /ROW2 -> /ROW4
- U1 pad 53: /ROW3 -> /ROW5
- U1 pad 55: /ROW5 -> /EN5_B
- U1 pad 56: /ROW6 -> /EN6_A
- U1 pad 57: unconnected-(U1-PB5-Pad57) -> /EN6_B
- U1 pad 61: unconnected-(U1-PB8-Pad61) -> /EN7_A
- U1 pad 62: unconnected-(U1-PB9-Pad62) -> /EN7_B
- WP14 pad 1: /COL1 -> /COL4
- WP22 pad 1: /COL2 -> /COL4
- X1 pad 3: Net-(U1-PF1) -> Net-(C7-Pad2)
Other:
- board outline added: 166.8 x 77.8 mm
- copper layers 2 -> 4

Commit message: update
Parts:
- removed C11, C12, C13, C14, C15, C16, C17, C18, C47, C53, C54: 100nF-CER-25V-0402, Capacitor_SMD:C_0402_1005Metric
- removed C19, C20: ~, Capacitor_SMD:C_0402_1005Metric
- removed C50, C51: c=1u, Capacitor_SMD:C_0805_2012Metric
- removed C52: c=4.7u, Capacitor_SMD:C_0805_2012Metric
- removed C55: c=100u, Capacitor_SMD:CP_Elec_6.3x5.9
- removed J4: USB_A, CONN-USB:GSB12121RSKHR
- removed R13, R14, R15, R16, R17, R18: 100kR-SMD-100mW-0603, Resistor_SMD:R_0603_1608Metric
- removed R19: r=49.9k, Resistor_SMD:R_0603_1608Metric
- removed R4: 12kR-SMD-100mW-0603, Resistor_SMD:R_0603_1608Metric
- removed U2: USB2512B, Package_DFN_QFN:QFN-36-1EP_6x6mm_P0.5mm_EP3.7x3.7mm_ThermalVias
- removed U4: ~, SOT-SMD:SOT-23-6
- removed X2: 24MHz, Crystal:Crystal_SMD_EuroQuartz_MT-4Pin_3.2x2.5mm
- D1, D2, D3, J3, L1, LF1, LF2: moved to B.Cu
- moved D12 318.0 mm to (41.3, 16.9)
- moved D13 318.0 mm to (41.3, 20.2)
- moved D4 318.0 mm to (29.7, 16.9)
- moved D5 318.0 mm to (29.7, 20.2)
- moved D6 318.0 mm to (29.7, 23.6)
- moved D7 318.0 mm to (29.7, 26.9)
- moved D10 318.0 mm to (35.5, 23.6)
- moved D11 318.0 mm to (35.5, 26.9)
- moved D8 318.0 mm to (35.5, 16.9)
- moved D9 318.0 mm to (35.5, 20.2)
- moved WP1 317.4 mm to (15.2, 29.7)
- moved WP10 317.4 mm to (23.8, 29.7)
- moved WP11 317.4 mm to (23.8, 32.6)
- moved WP12 317.4 mm to (23.8, 35.4)
- moved WP2 317.4 mm to (15.2, 32.6)
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Connections:
- C1 pad 1: Net-(U1-VDDA) -> /+3.3V
- C10 pad 1: +3.3V -> /+3.3V
- C2 pad 1: Net-(U1-VDDA) -> /+3.3V
- C21 pad 1: Net-(LED1-VDD) -> /LEDs/+5V
- C22 pad 1: Net-(LED2-VDD) -> /LEDs/+5V
- C23 pad 1: Net-(LED3-VDD) -> /LEDs/+5V
- C24 pad 1: Net-(LED4-VDD) -> /LEDs/+5V
- C25 pad 1: Net-(LED5-VDD) -> /LEDs/+5V
- C26 pad 1: Net-(LED6-VDD) -> /LEDs/+5V
- C27 pad 1: Net-(LED7-VDD) -> /LEDs/+5V
- C28 pad 1: Net-(LED8-VDD) -> /LEDs/+5V
- C29 pad 1: Net-(LED9-VDD) -> /LEDs/+5V
- C3 pad 1: Net-(U1-VDDA) -> /+3.3V
- C30 pad 1: Net-(LED10-VDD) -> /LEDs/+5V
- C31 pad 1: Net-(LED11-VDD) -> /LEDs/+5V
- C32 pad 1: Net-(LED12-VDD) -> /LEDs/+5V
- C33 pad 1: Net-(LED13-VDD) -> /LEDs/+5V
- C34 pad 1: Net-(LED14-VDD) -> /LEDs/+5V
- C35 pad 1: Net-(LED15-VDD) -> /LEDs/+5V
- C36 pad 1: Net-(LED16-VDD) -> /LEDs/+5V
- C37 pad 1: Net-(LED17-VDD) -> /LEDs/+5V
- C38 pad 1: Net-(LED18-VDD) -> /LEDs/+5V
- C39 pad 1: Net-(LED19-VDD) -> /LEDs/+5V
- C4 pad 1: Net-(U1-VDDA) -> /+3.3V
- C40 pad 1: Net-(LED20-VDD) -> /LEDs/+5V
- C41 pad 1: Net-(LED21-VDD) -> /LEDs/+5V
- C42 pad 1: Net-(LED22-VDD) -> /LEDs/+5V
- C48 pad 1: Net-(U1-VDDA) -> /+3.3V
- C49 pad 1: Net-(U1-VDDA) -> /+3.3V
- C5 pad 1: Net-(U1-VDDA) -> /+3.3V
- C9 pad 1: Net-(U3-VIN) -> /+5V
- ENC1 pad 2: Net-(ENC1-B) -> ~
- ENC1 pad 3: ~ -> Net-(ENC1-B)
- ENC2 pad 2: Net-(ENC2-B) -> ~
- ENC2 pad 3: ~ -> Net-(ENC2-B)
- ENC3 pad 2: Net-(ENC3-B) -> ~
- ENC3 pad 3: ~ -> Net-(ENC3-B)
- ENC4 pad 2: Net-(ENC4-B) -> ~
- ENC4 pad 3: ~ -> Net-(ENC4-B)
- J2 pad 9: Net-(J2-3.3V) -> /+3.3V
- J3 pad 0: (no net) -> Net-(D1-A1)
- J5 pad 1: Net-(J5-Pad1) -> /+5V
- J6 pad 6: Net-(J6-Pad6) -> /+5V
- J6 pad 8: Net-(J6-Pad8) -> /+3.3V
- L1 pad 1: /D+ -> /D-
- L1 pad 2: /USB_D+ -> /USB_MCU_D-
- L1 pad 3: /USB_D- -> /USB_MCU_D+
- L1 pad 4: /D- -> /D+
- LED1 pad 1: Net-(LED1-VDD) -> /LEDs/+5V
- LED10 pad 1: Net-(LED10-VDD) -> /LEDs/+5V
- LED11 pad 1: Net-(LED11-VDD) -> /LEDs/+5V
- LED12 pad 1: Net-(LED12-VDD) -> /LEDs/+5V
- LED13 pad 1: Net-(LED13-VDD) -> /LEDs/+5V
- LED14 pad 1: Net-(LED14-VDD) -> /LEDs/+5V
- LED15 pad 1: Net-(LED15-VDD) -> /LEDs/+5V
- LED16 pad 1: Net-(LED16-VDD) -> /LEDs/+5V
- LED17 pad 1: Net-(LED17-VDD) -> /LEDs/+5V
- LED18 pad 1: Net-(LED18-VDD) -> /LEDs/+5V
- LED19 pad 1: Net-(LED19-VDD) -> /LEDs/+5V
- LED2 pad 1: Net-(LED2-VDD) -> /LEDs/+5V
- LED20 pad 1: Net-(LED20-VDD) -> /LEDs/+5V
- LED21 pad 1: Net-(LED21-VDD) -> /LEDs/+5V
- LED22 pad 1: Net-(LED22-VDD) -> /LEDs/+5V
- LED3 pad 1: Net-(LED3-VDD) -> /LEDs/+5V
- LED4 pad 1: Net-(LED4-VDD) -> /LEDs/+5V
- LED5 pad 1: Net-(LED5-VDD) -> /LEDs/+5V
- LED6 pad 1: Net-(LED6-VDD) -> /LEDs/+5V
- LED7 pad 1: Net-(LED7-VDD) -> /LEDs/+5V
- LED8 pad 1: Net-(LED8-VDD) -> /LEDs/+5V
- LED9 pad 1: Net-(LED9-VDD) -> /LEDs/+5V
- LF1 pad 2: Net-(LF1-Pad2) -> /+5V
- R1 pad 1: Net-(R1-Pad1) -> /+3.3V
- R11 pad 1: Net-(R11-Pad1) -> /LEDs/+3.3V
- R12 pad 1: Net-(R11-Pad1) -> /LEDs/+3.3V
- R23 pad 1: Net-(R23-Pad1) -> /LEDs/+3.3V
- R24 pad 1: Net-(R23-Pad1) -> /LEDs/+3.3V
- R27 pad 1: Net-(R27-Pad1) -> /LEDs/+3.3V
- R28 pad 1: Net-(R27-Pad1) -> /LEDs/+3.3V
- R3 pad 1: Net-(U3-VIN) -> /+5V
- R33 pad 1: Net-(R33-Pad1) -> /LEDs/+3.3V
- R34 pad 1: Net-(R34-Pad1) -> /LEDs/+3.3V
- R35 pad 1: Net-(R33-Pad1) -> /LEDs/+3.3V
- R36 pad 1: Net-(R34-Pad1) -> /LEDs/+3.3V
- R39 pad 1: Net-(R39-Pad1) -> /+3.3V
- R40 pad 1: Net-(R39-Pad1) -> /+3.3V
- R43 pad 1: Net-(R43-Pad1) -> /+3.3V
- R44 pad 1: Net-(R43-Pad1) -> /+3.3V
- R5 pad 1: Net-(R5-Pad1) -> /LEDs/+3.3V
- R6 pad 1: Net-(R5-Pad1) -> /LEDs/+3.3V
- U1 pad 13: Net-(U1-VDDA) -> /+3.3V
- U1 pad 19: Net-(U1-VDDA) -> /+3.3V
- U1 pad 32: Net-(U1-VDDA) -> /+3.3V
- U1 pad 48: Net-(U1-VDDA) -> /+3.3V
- U1 pad 64: Net-(U1-VDDA) -> /+3.3V
- U3 pad 1: Net-(U3-VIN) -> /+5V
- U3 pad 5: +3.3V -> /+3.3V
- WP1 pad 1: Net-(WP1-Pad1) -> /+3.3V
- WP11 pad 1: Net-(WP11-Pad1) -> /+3.3V
- WP5 pad 1: Net-(WP1-Pad1) -> /+3.3V
- WP8 pad 1: Net-(WP11-Pad1) -> /+3.3V
Routing:
- net /~{nRST}: track 0.00 -> 40.7 mm
- net /DBG_TX: track 0.00 -> 21.7 mm
- net /DBG_RX: track 0.00 -> 19.8 mm
- net /SWDIO: track 0.00 -> 17.9 mm
- net /SWCLK: track 0.00 -> 15.8 mm
- net /+3.3V: track 0.00 -> 11.5 mm
- net /USB_MCU_D-: track 0.00 -> 8.22 mm, vias 0 -> 1
- net /USB_MCU_D+: track 0.00 -> 7.43 mm, vias 0 -> 1
- net Net-(U1-PF1): track 0.00 -> 6.85 mm
- net Net-(D1-A2): track 0.00 -> 6.16 mm
- net Net-(U1-PF0): track 0.00 -> 5.34 mm
- net /D+: track 0.00 -> 3.90 mm
- net /D-: track 0.00 -> 3.90 mm
- net Net-(ENC1-A): track 0.00 -> 3.44 mm
- net Net-(ENC2-B): track 0.00 -> 3.43 mm
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- added copper zone on B.Cu, net Net-(D1-A1)
- added copper zone on In2.Cu, net Net-(D1-A1)
- added copper zone on F.Cu, net ~
Other:
- outline, holes or cut-outs redrawn
