File: GT-Wheel-Main-PCB/GT-Wheel.kicad_sch (KiCad schematic)
At the start: 57 parts, among them J2 TC2050, J3 0532610471, J5 0532610871, J6 0532610871, U1 STM32F303RETx, U3 AP2112K-3.3, X1 32MHz

Commit message: update
Connections:
- net +3.3V: now also C1.1, C2.1, C3.1, C4.1, C48.1, C49.1, C5.1, J2.9 (3.3V), J6.8, R1.1, R39.1, R40.1, R43.1, R44.1, U1.13 (VDDA), U1.19 (VDD), U1.32 (VDD), U1.48 (VDD), U1.64 (VDD), WP1.1, WP11.1, WP5.1, WP8.1
- net D+: now also L1.4; no longer L1.1
- net D-: now also L1.1; no longer L1.4
- net USB_MCU_D+: now also L1.3; no longer L1.2
- net USB_MCU_D-: now also L1.2; no longer L1.3
- net +5V: now reaches C9.1, R3.1, U3.1 (VIN)
- net +5V: now also J5.1, J6.6, LF1.2
Changed lines of the file:
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@@
     (stroke (width 0) (type default))
   )
+  (wire (pts (xy 20.32 66.04) (xy 20.32 68.58))
+    (stroke (width 0) (type default))
+  )
   (wire (pts (xy 35.56 114.3) (xy 35.56 121.92))
     (stroke (width 0) (type default))
@@
     (effects (font (size 1.27 1.27)) (justify right bottom))
   )
+  (label "+5V" (at 86.36 185.42 0) (fields_autoplaced)
+    (effects (font (size 1.27 1.27)) (justify left bottom))
+  )
   (label "D-" (at 116.84 132.08 0) (fields_autoplaced)
     (effects (font (size 1.27 1.27)) (justify left bottom))
@@
     (effects (font (size 1.27 1.27)) (justify left bottom))
   )
+  (label "+3.3V" (at 152.4 25.4 90) (fields_autoplaced)
+    (effects (font (size 1.27 1.27)) (justify left bottom))
+  )
   (label "SWCLK" (at 99.06 73.66 0) (fields_autoplaced)
     (effects (font (size 1.27 1.27)) (justify left bottom))
@@
     (effects (font (size 1.27 1.27)) (justify left bottom))
   )
+  (label "+3.3V" (at 127 182.88 90) (fields_autoplaced)
+    (effects (font (size 1.27 1.27)) (justify left bottom))
+  )
   (label "NAV1_ENC_B" (at 48.26 68.58 0) (fields_autoplaced)
     (effects (font (size 1.27 1.27)) (justify left bottom))
   )
+  (label "+3.3V" (at 152.4 60.96 90) (fields_autoplaced)
+    (effects (font (size 1.27 1.27)) (justify left bottom))
+  )
   (label "LED_DIN" (at 228.6 17.78 0) (fields_autoplaced)
     (effects (font (size 1.27 1.27)) (justify left bottom))
@@
     (effects (font (size 1.27 1.27)) (justify left bottom))
   )
+  (label "+5V" (at 149.86 127 0) (fields_autoplaced)
+    (effects (font (size 1.27 1.27)) (justify left bottom))
+  )
   (label "COL1" (at 185.42 20.32 270) (fields_autoplaced)
     (effects (font (size 1.27 1.27)) (justify right bottom))
@@
     (effects (font (size 1.27 1.27)) (justify left bottom))
   )
+  (label "+3.3V" (at 20.32 68.58 90) (fields_autoplaced)
+    (effects (font (size 1.27 1.27)) (justify left bottom))
+  )
   (label "SHIFT_UP" (at 116.84 187.96 0) (fields_autoplaced)
     (effects (font (size 1.27 1.27)) (justify left bottom))
@@
     (effects (font (size 1.27 1.27)) (justify left bottom))
   )
+  (label "+3.3V" (at 66.04 22.86 0) (fields_autoplaced)
+    (effects (font (size 1.27 1.27)) (justify left bottom))
+  )
+  (label "+5V" (at 25.4 111.76 0) (fields_autoplaced)
+    (effects (font (size 1.27 1.27)) (justify left bottom))
+  )
   (label "COL4" (at 193.04 20.32 270) (fields_autoplaced)
     (effects (font (size 1.27 1.27)) (justify right bottom))
@@
     (effects (font (size 1.27 1.27)) (justify left bottom))
   )
+  (label "+3.3V" (at 30.48 20.32 90) (fields_autoplaced)
+    (effects (font (size 1.27 1.27)) (justify left bottom))
+  )
+  (label "+3.3V" (at 86.36 190.5 0) (fields_autoplaced)
+    (effects (font (size 1.27 1.27)) (justify left bottom))
+  )
   (label "EN3_B" (at 88.9 175.26 0) (fields_autoplaced)
     (effects (font (size 1.27 1.27)) (justify left bottom))
@@
     (effects (font (size 1.27 1.27)) (justify left bottom))
   )
+  (label "+5V" (at 88.9 149.86 0) (fields_autoplaced)
+    (effects (font (size 1.27 1.27)) (justify left bottom))
+  )
   (label "USB_MCU_D-" (at 99.06 66.04 0) (fields_autoplaced)
     (effects (font (size 1.27 1.27)) (justify left bottom))
@@
     (effects (font (size 1.27 1.27)) (justify left bottom))
   )
+  (label "+3.3V" (at 53.34 111.76 0) (fields_autoplaced)
+    (effects (font (size 1.27 1.27)) (justify left bottom))
+  )
   (label "D+" (at 116.84 129.54 0) (fields_autoplaced)
     (effects (font (size 1.27 1.27)) (justify left bottom))
@@
     (effects (font (size 1.27 1.27)) (justify left bottom))
   )
+  (label "+3.3V" (at 157.48 182.88 90) (fields_autoplaced)
+    (effects (font (size 1.27 1.27)) (justify left bottom))
+  )
   (symbol (lib_id "POWER:LOGIC_GND") (at 58.42 119.38 0) (unit 1)
     (in_bom yes) (on_board yes) (dnp no) (fields_autoplaced)
@@
     )
   )
-  (symbol (lib_id "power:+3.3V") (at 58.42 109.22 0) (unit 1)
-    (in_bom yes) (on_board yes) (dnp no) (fields_autoplaced)
-    (property "Reference" "#PWR015" (at 58.42 113.03 0)
+  (symbol (lib_id "POWER:+3.3V") (at 58.42 109.22 0) (unit 1)
+    (in_bom yes) (on_board yes) (dnp no)
+    (property "Reference" "#PWR05" (at 55.499 110.109 0)
       (effects (font (size 1.27 1.27)) hide)
     )
-    (property "Value" "+3.3V" (at 58.42 104.14 0)
+    (property "Value" "+3.3V" (at 58.42 105.41 0)
       (effects (font (size 1.27 1.27)))
     )
-    (property "Footprint" "" (at 58.42 109.22 0)
+    (property "Footprint" "" (at 58.801 106.68 0)
       (effects (font (size 1.27 1.27)) hide)
     )
-    (property "Datasheet" "" (at 58.42 109.22 0)
+    (property "Datasheet" "" (at 58.801 106.68 0)
       (effects (font (size 1.27 1.27)) hide)
     )
-    (pin "1")
+    (pin "~")
     (instances
       (project "GT-Wheel"
         (path "/be9b0bd3-2348-472d-a590-21f5b0c33bd7"
-          (reference "#PWR015") (unit 1)
+          (reference "#PWR05") (unit 1)
         )
       )
@@
     )
   )
-  (symbol (lib_id "POWER:+3.3V") (at 20.32 68.58 0) (unit 1)
+  (symbol (lib_id "POWER:+3.3V") (at 20.32 66.04 0) (unit 1)
     (in_bom yes) (on_board yes) (dnp no)
-    (property "Reference" "#PWR0112" (at 17.399 69.469 0)
+    (property "Reference" "#PWR0112" (at 17.399 66.929 0)
       (effects (font (size 1.27 1.27)) hide)
     )
-    (property "Value" "+3.3V" (at 20.32 64.77 0)
+    (property "Value" "+3.3V" (at 20.32 62.23 0)
       (effects (font (size 1.27 1.27)))
     )
-    (property "Footprint" "" (at 20.701 66.04 0)
+    (property "Footprint" "" (at 20.701 63.5 0)
       (effects (font (size 1.27 1.27)) hide)
     )
-    (property "Datasheet" "" (at 20.701 66.04 0)
+    (property "Datasheet" "" (at 20.701 63.5 0)
       (effects (font (size 1.27 1.27)) hide)
     )
@@
     )
   )
-  (symbol (lib_id "IND-SMD-CHOKE:DLW21HN900SQ2L") (at 142.24 132.08 0) (unit 1)
+  (symbol (lib_id "IND-SMD-CHOKE:DLW21HN900SQ2L") (at 142.24 132.08 0) (mirror x) (unit 1)
     (in_bom yes) (on_board yes) (dnp no)
-    (property "Reference" "L1" (at 142.24 128.27 0)
+    (property "Reference" "L1" (at 142.24 135.89 0)
       (effects (font (size 1.27 1.27)))
     )
-    (property "Value" "DLW21HN900SQ2L" (at 142.24 135.89 0)
+    (property "Value" "DLW21HN900SQ2L" (at 142.24 128.27 0)
       (effects (font (size 1.27 1.27)))
     )
-    (property "Footprint" "IND-SMD-CHOKE:FIL_DLW21HN900SQ2L" (at 141.097 124.714 0)
+    (property "Footprint" "IND-SMD-CHOKE:FIL_DLW21HN900SQ2L" (at 141.097 139.446 0)
       (effects (font (size 1.27 1.27)) hide)
     )
-    (property "Datasheet" "https://www.murata.com/~/media/webrenewal/products/emiconfun/mail/2013/06/28/en-20130628/l0114s0133dlw21h.ashx" (at 141.097 124.714 0)
+    (property "Datasheet" "https://www.murata.com/~/media/webrenewal/products/emiconfun/mail/2013/06/28/en-20130628/l0114s0133dlw21h.ashx" (at 141.097 139.446 0)
       (effects (font (size 1.27 1.27)) hide)
     )
